File: ampere/ampere.kicad_pcb (KiCad board)
At the start: 4 copper layers, 100 x 65 mm, 210 parts, among them J1 USB_C_Receptacle, J2 Channel 1, J3 Channel 2, J5 Conn_02x13_Odd_Even, Q1 BSC040N08NS5, Q10 AO4485, Q12 BSC040N08NS5, Q2 CSD25481F4, Q3 CSD25481F4, Q4 CSD13381F4, Q5 CSD13381F4, Q6 CSD17484F4, Q7 CSD17484F4, Q8 CSD18543Q3A, Q9 AO4485, U11 MCP4725xxx-xCH, U13 INA238, U14 INA238, U15 MCP4725xxx-xCH, U18 INA238, U19 INA238, U2 STM32G474RETx, U21 LM74502DDFR, U22 LMR36520ADDA, U23 TPS7A91, U3 TPS26750SRSMR, U4 TPD4S480RUKR, U5 CAT24C256, U6 TPS55289, U7 MIC29302WU, U8 TPS55289, U9 MIC29302WU, Y1 25 MHZ, Y2 32.768 KHZ

Commit message: add bottom traces to tps26750
Parts:
- added J1: USB_C_Receptacle, DX07S024JJ2R1300:JAE_DX07S024JJ2R1300, F.Cu at (227.5, 84.4)
Routing:
- net /GPIO3: track 2.45 -> 16.5 mm
- net /GPIO2: track 3.38 -> 16.6 mm
- net Net-(Q8-G): track 0.97 -> 8.38 mm, vias 1 -> 2
- net Net-(U21-OV): track 0.00 -> 2.55 mm
