File: ampere/system_power.kicad_sch (KiCad schematic)
At the start: 19 parts, among them U22 LMR36510ADDA, U23 TPS7A91

Commit message: add lmr36520 layout, expand board size to accomedate
Parts:
- C122, C123: value 22uF -> 4.7uF
- C124: value 22uF -> 220nF
- C129: footprint Capacitor_SMD:C_0603_1608Metric -> Capacitor_SMD:C_0402_1005Metric
- R81: value 38.3K -> 38.2K
- U22: value LMR36510ADDA -> LMR36520ADDA
Other:
- note added: "5V-28V -> 3.6V"
- title: (none) -> System Power Rails
- moved on the sheet: C118, C119, C120, C121, C122, C123, C124, C125, C126, C127, C128, C129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

Commit message: implement tps26750 and tpd4s480
Parts:
- R82, R83: footprint Resistor_SMD:R_0603_1608Metric -> Capacitor_SMD:C_0402_1005Metric
Changed lines of the file:
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@@
 			)
 		)
-		(property "Footprint" "Resistor_SMD:R_0603_1608Metric"
+		(property "Footprint" "Capacitor_SMD:C_0402_1005Metric"
 			(at 206.375 102.87 0)
 			(hide yes)
@@
 			)
 		)
-		(property "Footprint" "Resistor_SMD:R_0603_1608Metric"
+		(property "Footprint" "Capacitor_SMD:C_0402_1005Metric"
 			(at 206.375 97.79 0)
 			(hide yes)

Commit message: finalize display interconnect corridor
Parts:
- U23: footprint Package_DFN_QFN:Texas_S-PDSO-N10_EP1.2x2mm_ThermalVias -> Package_DFN_QFN:Texas_S-PDSO-N10_EP1.2x2mm
Changed lines of the file:
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@@
 			)
 		)
-		(property "Footprint" "Package_DFN_QFN:Texas_S-PDSO-N10_EP1.2x2mm_ThermalVias"
+		(property "Footprint" "Package_DFN_QFN:Texas_S-PDSO-N10_EP1.2x2mm"
 			(at 190.5 101.6 0)
 			(hide yes)
